File: KiCAD/ruler.kicad_pcb (KiCad board)
At the start: 2 copper layers, 100 x 32 mm, 70 parts, among them J1 ICP6, U1 ATtiny85V-10SU

Commit message: update
Parts:
- removed Re: 330, Resistor_SMD:R_0402_1005Metric
- removed tp1: ⌀2.5, TestPoint:TestPoint_Pad_D2.5mm
- added R4: 0805, Resistor_SMD:R_0805_2012Metric, B.Cu at (123.2, 114.9)
- added TP9: 0201, TestPoint:TestPoint_Pad_D1.0mm, F.Cu at (118.1, 123.8)
- R1: value 330 -> 0201; footprint Resistor_SMD:R_1206_3216Metric_Pad1.42x1.75mm_HandSolder -> Resistor_SMD:R_0201_0603Metric; moved to B.Cu
- R10: value 0201 -> 0805; footprint Resistor_SMD:R_0201_0603Metric -> Resistor_SMD:R_0805_2012Metric
- R11: value 0201 -> 1206; footprint Resistor_SMD:R_0201_0603Metric -> Resistor_SMD:R_1206_3216Metric
- R12, R6: value 0201 -> 2512; footprint Resistor_SMD:R_0201_0603Metric -> Resistor_SMD:R_2512_6332Metric
- R15, R19: value 0402 -> 0603; footprint Resistor_SMD:R_0402_1005Metric -> Resistor_SMD:R_0603_1608Metric
- R16: value 0402 -> 0805; footprint Resistor_SMD:R_0402_1005Metric -> Resistor_SMD:R_0805_2012Metric
- R17: value 0402 -> 1206; footprint Resistor_SMD:R_0402_1005Metric -> Resistor_SMD:R_1206_3216Metric
- R2: value 330 -> 0402; footprint Resistor_SMD:R_0805_2012Metric_Pad1.15x1.40mm_HandSolder -> Resistor_SMD:R_0402_1005Metric; moved to B.Cu
- R20: value 0603 -> 0805; footprint Resistor_SMD:R_0603_1608Metric -> Resistor_SMD:R_0805_2012Metric
- R21, R22: value 0603 -> 0201; footprint Resistor_SMD:R_0603_1608Metric -> Resistor_SMD:R_0201_0603Metric
- R23: value 0603 -> 0402; footprint Resistor_SMD:R_0603_1608Metric -> Resistor_SMD:R_0402_1005Metric
- R24: value 0603HS -> 0402; footprint Resistor_SMD:R_0603_1608Metric_Pad1.05x0.95mm_HandSolder -> Resistor_SMD:R_0402_1005Metric
- R25: value 0603HS -> 0201; footprint Resistor_SMD:R_0603_1608Metric_Pad1.05x0.95mm_HandSolder -> Resistor_SMD:R_0201_0603Metric
- R26: footprint Resistor_SMD:R_0603_1608Metric_Pad1.05x0.95mm_HandSolder -> Resistor_SMD:R_0603_1608Metric_Pad0.98x0.95mm_HandSolder
- R27: value 0603HS -> 0805HS; footprint Resistor_SMD:R_0603_1608Metric_Pad1.05x0.95mm_HandSolder -> Resistor_SMD:R_0805_2012Metric_Pad1.20x1.40mm_HandSolder
- R28: value 0805 -> 1206HS; footprint Resistor_SMD:R_0805_2012Metric -> Resistor_SMD:R_1206_3216Metric_Pad1.30x1.75mm_HandSolder
- R29: value 0805 -> 2512HS; footprint Resistor_SMD:R_0805_2012Metric -> Resistor_SMD:R_2512_6332Metric_Pad1.40x3.35mm_HandSolder
- R3: value 330 -> 0603; footprint Resistor_SMD:R_0603_1608Metric_Pad1.05x0.95mm_HandSolder -> Resistor_SMD:R_0603_1608Metric; moved to B.Cu
- R30: value 0805 -> 0201; footprint Resistor_SMD:R_0805_2012Metric -> Resistor_SMD:R_0201_0603Metric
- R31: value 0805 -> 0603HS; footprint Resistor_SMD:R_0805_2012Metric -> Resistor_SMD:R_0603_1608Metric_Pad0.98x0.95mm_HandSolder
- R32: footprint Resistor_SMD:R_0805_2012Metric_Pad1.15x1.40mm_HandSolder -> Resistor_SMD:R_0805_2012Metric_Pad1.20x1.40mm_HandSolder
- R33: value 0805HS -> 1206HS; footprint Resistor_SMD:R_0805_2012Metric_Pad1.15x1.40mm_HandSolder -> Resistor_SMD:R_1206_3216Metric_Pad1.30x1.75mm_HandSolder
- R34: value 0805HS -> 2512HS; footprint Resistor_SMD:R_0805_2012Metric_Pad1.15x1.40mm_HandSolder -> Resistor_SMD:R_2512_6332Metric_Pad1.40x3.35mm_HandSolder
- R35: value 0805HS -> 0201; footprint Resistor_SMD:R_0805_2012Metric_Pad1.15x1.40mm_HandSolder -> Resistor_SMD:R_0201_0603Metric
- R36: value 1206 -> 0603HS; footprint Resistor_SMD:R_1206_3216Metric -> Resistor_SMD:R_0603_1608Metric_Pad0.98x0.95mm_HandSolder
- R37: value 1206 -> 0805HS; footprint Resistor_SMD:R_1206_3216Metric -> Resistor_SMD:R_0805_2012Metric_Pad1.20x1.40mm_HandSolder
- R38: value 1206 -> 1206HS; footprint Resistor_SMD:R_1206_3216Metric -> Resistor_SMD:R_1206_3216Metric_Pad1.30x1.75mm_HandSolder
- R39: value 1206HS -> 0603HS; footprint Resistor_SMD:R_1206_3216Metric_Pad1.42x1.75mm_HandSolder -> Resistor_SMD:R_0603_1608Metric_Pad0.98x0.95mm_HandSolder
- R40: value 1206HS -> 0805HS; footprint Resistor_SMD:R_1206_3216Metric_Pad1.42x1.75mm_HandSolder -> Resistor_SMD:R_0805_2012Metric_Pad1.20x1.40mm_HandSolder
- R41: value 1206HS -> 330; moved to F.Cu
- R42: value 2512 -> 330; footprint Resistor_SMD:R_2512_6332Metric -> Resistor_SMD:R_0805_2012Metric_Pad1.20x1.40mm_HandSolder; moved to F.Cu
- R43: value 2512 -> 330; footprint Resistor_SMD:R_2512_6332Metric -> Resistor_SMD:R_0603_1608Metric_Pad0.98x0.95mm_HandSolder; moved to F.Cu
- R44: value 2512HS -> 330; footprint Resistor_SMD:R_2512_6332Metric_Pad1.52x3.35mm_HandSolder -> Resistor_SMD:R_0402_1005Metric; moved to F.Cu
- R45: value 2512HS -> 330; footprint Resistor_SMD:R_2512_6332Metric_Pad1.52x3.35mm_HandSolder -> Resistor_SMD:R_0201_0603Metric; moved to F.Cu
- R5: value 330 -> 1206; footprint Resistor_SMD:R_0201_0603Metric -> Resistor_SMD:R_1206_3216Metric; moved to B.Cu
- R8: value 0201 -> 0402; footprint Resistor_SMD:R_0201_0603Metric -> Resistor_SMD:R_0402_1005Metric
- R9: value 0201 -> 0603; footprint Resistor_SMD:R_0201_0603Metric -> Resistor_SMD:R_0603_1608Metric
- TP1: value 1206 -> ⌀1.0; moved to B.Cu
- TP2: value 0805 -> ⌀1.5; footprint TestPoint:TestPoint_Pad_D1.0mm -> TestPoint:TestPoint_Pad_D1.5mm; moved to B.Cu
- TP3: value 0603 -> ⌀2.0; footprint TestPoint:TestPoint_Pad_D1.0mm -> TestPoint:TestPoint_Pad_D2.0mm; moved to B.Cu
- TP4: value 0402 -> ⌀2.5; footprint TestPoint:TestPoint_Pad_D1.0mm -> TestPoint:TestPoint_Pad_D2.5mm; moved to B.Cu
- TP5: value 0201 -> 1206
- TP6: value ⌀1.0 -> 0805; moved to F.Cu
- TP7: value ⌀1.5 -> 0603; footprint TestPoint:TestPoint_Pad_D1.5mm -> TestPoint:TestPoint_Pad_D1.0mm; moved to F.Cu
- TP8: value ⌀2.0 -> 0402; footprint TestPoint:TestPoint_Pad_D2.0mm -> TestPoint:TestPoint_Pad_D1.0mm; moved to F.Cu
- moved TP1 40.5 mm to (156.8, 125.7), turned to 180 degrees
- moved TP6 39.5 mm to (118.1, 115.6), turned to 180 degrees
- moved TP2 36.4 mm to (153.7, 125.7), turned to 180 degrees
- moved TP7 34.7 mm to (118.1, 118.7), turned to 180 degrees
- moved TP3 31.4 mm to (149.2, 125.7), turned to 180 degrees
- moved TP8 30.1 mm to (118.1, 121.3), turned to 180 degrees
- moved R41 28.7 mm to (121.3, 111.8), turned to 180 degrees
- moved R45 27.0 mm to (121.3, 123.8), turned to 180 degrees
- moved R36 26.4 mm to (97.2, 111.8)
- moved TP4 25.9 mm to (144.1, 125.7), turned to 180 degrees
- moved R37 20.7 mm to (97.2, 114.9)
- moved R35 19.8 mm to (109.9, 105.4)
- moved R38 19.1 mm to (93.3, 118.7)
- moved R28 18.6 mm to (104.8, 118.7)
- moved R6 18.5 mm to (121.3, 123.8)
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Connections:
- D1 pad 2: Net-(D1-Pad2) -> Net-(D1-A)
- D2 pad 2: Net-(D2-Pad2) -> Net-(D2-A)
- D3 pad 2: Net-(D3-Pad2) -> Net-(D3-A)
- D4 pad 2: Net-(D4-Pad2) -> Net-(D4-A)
- D5 pad 2: Net-(D5-Pad2) -> Net-(D5-A)
- R1 pad 1: Net-(D1-Pad2) -> unconnected-(R1-Pad1)
- R1 pad 2: 1206 -> unconnected-(R1-Pad2)
- R10 pad 1: Net-(R10-Pad1) -> unconnected-(R10-Pad1)
- R10 pad 2: Net-(R10-Pad2) -> unconnected-(R10-Pad2)
- R11 pad 1: Net-(R11-Pad1) -> unconnected-(R11-Pad1)
- R11 pad 2: Net-(R11-Pad2) -> unconnected-(R11-Pad2)
- R12 pad 1: Net-(R12-Pad1) -> unconnected-(R12-Pad1)
- R12 pad 2: Net-(R12-Pad2) -> unconnected-(R12-Pad2)
- R13 pad 1: Net-(R13-Pad1) -> unconnected-(R13-Pad1)
- R13 pad 2: Net-(R13-Pad2) -> unconnected-(R13-Pad2)
- R14 pad 1: Net-(R14-Pad1) -> unconnected-(R14-Pad1)
- R14 pad 2: Net-(R14-Pad2) -> unconnected-(R14-Pad2)
- R15 pad 1: Net-(R15-Pad1) -> unconnected-(R15-Pad1)
- R15 pad 2: Net-(R15-Pad2) -> unconnected-(R15-Pad2)
- R16 pad 1: Net-(R16-Pad1) -> unconnected-(R16-Pad1)
- R16 pad 2: Net-(R16-Pad2) -> unconnected-(R16-Pad2)
- R17 pad 1: Net-(R17-Pad1) -> unconnected-(R17-Pad1)
- R17 pad 2: Net-(R17-Pad2) -> unconnected-(R17-Pad2)
- R18 pad 1: Net-(R18-Pad1) -> unconnected-(R18-Pad1)
- R18 pad 2: Net-(R18-Pad2) -> unconnected-(R18-Pad2)
- R19 pad 1: Net-(R19-Pad1) -> unconnected-(R19-Pad1)
- R19 pad 2: Net-(R19-Pad2) -> unconnected-(R19-Pad2)
- R2 pad 1: Net-(D2-Pad2) -> unconnected-(R2-Pad1)
- R2 pad 2: 0805 -> unconnected-(R2-Pad2)
- R20 pad 1: Net-(R20-Pad1) -> unconnected-(R20-Pad1)
- R20 pad 2: Net-(R20-Pad2) -> unconnected-(R20-Pad2)
- R21 pad 1: Net-(R21-Pad1) -> unconnected-(R21-Pad1)
- R21 pad 2: Net-(R21-Pad2) -> unconnected-(R21-Pad2)
- R22 pad 1: Net-(R22-Pad1) -> unconnected-(R22-Pad1)
- R22 pad 2: Net-(R22-Pad2) -> unconnected-(R22-Pad2)
- R23 pad 1: Net-(R23-Pad1) -> unconnected-(R23-Pad1)
- R23 pad 2: Net-(R23-Pad2) -> unconnected-(R23-Pad2)
- R24 pad 1: Net-(R24-Pad1) -> unconnected-(R24-Pad1)
- R24 pad 2: Net-(R24-Pad2) -> unconnected-(R24-Pad2)
- R25 pad 1: Net-(R25-Pad1) -> unconnected-(R25-Pad1)
- R25 pad 2: Net-(R25-Pad2) -> unconnected-(R25-Pad2)
- R26 pad 1: Net-(R26-Pad1) -> unconnected-(R26-Pad1)
- R26 pad 2: Net-(R26-Pad2) -> unconnected-(R26-Pad2)
- R27 pad 1: Net-(R27-Pad1) -> unconnected-(R27-Pad1)
- R27 pad 2: Net-(R27-Pad2) -> unconnected-(R27-Pad2)
- R28 pad 1: Net-(R28-Pad1) -> unconnected-(R28-Pad1)
- R28 pad 2: Net-(R28-Pad2) -> unconnected-(R28-Pad2)
- R29 pad 1: Net-(R29-Pad1) -> unconnected-(R29-Pad1)
- R29 pad 2: Net-(R29-Pad2) -> unconnected-(R29-Pad2)
- R3 pad 1: Net-(D3-Pad2) -> unconnected-(R3-Pad1)
- R3 pad 2: 0603 -> unconnected-(R3-Pad2)
- R30 pad 1: Net-(R30-Pad1) -> unconnected-(R30-Pad1)
- R30 pad 2: Net-(R30-Pad2) -> unconnected-(R30-Pad2)
- R31 pad 1: Net-(R31-Pad1) -> unconnected-(R31-Pad1)
- R31 pad 2: Net-(R31-Pad2) -> unconnected-(R31-Pad2)
- R32 pad 1: Net-(R32-Pad1) -> unconnected-(R32-Pad1)
- R32 pad 2: Net-(R32-Pad2) -> unconnected-(R32-Pad2)
- R33 pad 1: Net-(R33-Pad1) -> unconnected-(R33-Pad1)
- R33 pad 2: Net-(R33-Pad2) -> unconnected-(R33-Pad2)
- R34 pad 1: Net-(R34-Pad1) -> unconnected-(R34-Pad1)
- R34 pad 2: Net-(R34-Pad2) -> unconnected-(R34-Pad2)
- R35 pad 1: Net-(R35-Pad1) -> unconnected-(R35-Pad1)
- R35 pad 2: Net-(R35-Pad2) -> unconnected-(R35-Pad2)
- R36 pad 1: Net-(R36-Pad1) -> unconnected-(R36-Pad1)
- R36 pad 2: Net-(R36-Pad2) -> unconnected-(R36-Pad2)
- R37 pad 1: Net-(R37-Pad1) -> unconnected-(R37-Pad1)
- R37 pad 2: Net-(R37-Pad2) -> unconnected-(R37-Pad2)
- R38 pad 1: Net-(R38-Pad1) -> unconnected-(R38-Pad1)
- R38 pad 2: Net-(R38-Pad2) -> unconnected-(R38-Pad2)
- R39 pad 1: Net-(R39-Pad1) -> unconnected-(R39-Pad1)
- R39 pad 2: Net-(R39-Pad2) -> unconnected-(R39-Pad2)
- R40 pad 1: Net-(R40-Pad1) -> unconnected-(R40-Pad1)
- R40 pad 2: Net-(R40-Pad2) -> unconnected-(R40-Pad2)
- R41 pad 1: Net-(R41-Pad1) -> Net-(D1-A)
- R41 pad 2: Net-(R41-Pad2) -> 1206
- R42 pad 1: Net-(R42-Pad1) -> Net-(D2-A)
- R42 pad 2: Net-(R42-Pad2) -> 0805
- R43 pad 1: Net-(R43-Pad1) -> Net-(D3-A)
- R43 pad 2: Net-(R43-Pad2) -> 0603
- R44 pad 1: Net-(R44-Pad1) -> Net-(D4-A)
- R44 pad 2: Net-(R44-Pad2) -> 0402
- R45 pad 1: Net-(R45-Pad1) -> Net-(D5-A)
- R45 pad 2: Net-(R45-Pad2) -> 0201
- R5 pad 1: Net-(D5-Pad2) -> unconnected-(R5-Pad1)
- R5 pad 2: 0201 -> unconnected-(R5-Pad2)
- R6 pad 1: Net-(R6-Pad1) -> unconnected-(R6-Pad1)
- R6 pad 2: Net-(R6-Pad2) -> unconnected-(R6-Pad2)
- R7 pad 1: Net-(R7-Pad1) -> unconnected-(R7-Pad1)
- R7 pad 2: Net-(R7-Pad2) -> unconnected-(R7-Pad2)
- R8 pad 1: Net-(R8-Pad1) -> unconnected-(R8-Pad1)
- R8 pad 2: Net-(R8-Pad2) -> unconnected-(R8-Pad2)
- R9 pad 1: Net-(R9-Pad1) -> unconnected-(R9-Pad1)
- R9 pad 2: Net-(R9-Pad2) -> unconnected-(R9-Pad2)
- TP1 pad 1: 1206 -> unconnected-(TP1-Pad1)
- TP2 pad 1: 0805 -> unconnected-(TP2-Pad1)
- TP3 pad 1: 0603 -> unconnected-(TP3-Pad1)
- TP4 pad 1: 0402 -> unconnected-(TP4-Pad1)
- TP5 pad 1: 0201 -> 1206
- TP6 pad 1: Net-(TP6-Pad1) -> 0805
- TP7 pad 1: Net-(TP7-Pad1) -> 0603
- TP8 pad 1: Net-(TP8-Pad1) -> 0402
Routing:
- net +5V: track 70.0 -> 34.5 mm, vias 2 -> 1
- net 0201: track 24.2 -> 0.00 mm, vias 2 -> 0
- net 0402: track 23.9 -> 0.00 mm, vias 2 -> 0
- net 0603: track 64.3 -> 45.5 mm, vias 2 -> 0
- net 0805: track 57.6 -> 40.4 mm, vias 2 -> 0
- net 1206: track 52.1 -> 37.6 mm
- net Net-(D5-Pad2): track 6.73 -> 0.00 mm
- net Net-(D4-Pad2): track 6.14 -> 0.00 mm
- net Net-(D5-A): track 0.00 -> 5.16 mm
- net Net-(D4-A): track 0.00 -> 4.76 mm
- net Net-(D3-Pad2): track 4.71 -> 0.00 mm
- net Net-(D2-Pad2): track 4.31 -> 0.00 mm
- net Net-(D3-A): track 0.00 -> 4.02 mm
- net Net-(D2-A): track 0.00 -> 3.74 mm
- net Net-(D1-Pad2): track 2.79 -> 0.00 mm
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
Commit message: .
Parts:
- removed Logo1: SquashedFlyLogo, SquashedFly Logo:SquashedFly Logo
- added REF**: SquashedFlySilk, KiCad Footprints:SquashedFlySilk, F.Cu at (181.6, 123.8)
Routing:
- net 1206: track 37.6 -> 50.1 mm
- net GND: track 102.0 -> 91.6 mm
- net 0201: track 0.00 -> 2.86 mm
- net 0402: track 0.00 -> 2.67 mm
- net 0603: track 45.5 -> 47.8 mm
- net 0805: track 40.4 -> 42.6 mm
