File: KiCAD/ruler.kicad_sch (KiCad schematic)
At the start: 64 parts

Commit message: .
Parts:
- BT1: value (none) -> 3V Cell; footprint (none) -> Battery:BatteryHolder_Keystone_3002_1x2032
- C1: value (none) -> 0.1uF; footprint (none) -> Capacitor_SMD:C_0805_2012Metric_Pad1.15x1.40mm_HandSolder
- D1: value (none) -> 1206 Red; footprint (none) -> LED_SMD:LED_1206_3216Metric_Pad1.42x1.75mm_HandSolder
- D2: value (none) -> 0805 Orange; footprint (none) -> LED_SMD:LED_0805_2012Metric_Pad1.15x1.40mm_HandSolder
- D3: value (none) -> 0603 Yellow; footprint (none) -> LED_SMD:LED_0603_1608Metric_Pad1.05x0.95mm_HandSolder
- D4: value (none) -> 0402 Green; footprint (none) -> LED_SMD:LED_0402_1005Metric
- D5: value (none) -> 0201 Blue; footprint (none) -> LED_SMD:LED_0201_0603Metric
- J1: value (none) -> ICP6; footprint (none) -> Connector_PinHeader_2.54mm:PinHeader_2x03_P2.54mm_Vertical
- Logo1: value (none) -> SquashedFlyLogo; footprint (none) -> SquashedFly Logo:SquashedFly Logo
- R1: value (none) -> 330; footprint (none) -> Resistor_SMD:R_1206_3216Metric_Pad1.42x1.75mm_HandSolder
- R10, R11, R12, R13, R6, R7, R8, R9: value (none) -> 0201; footprint (none) -> Resistor_SMD:R_0201_0603Metric
- R14, R15, R16, R17, R18, R19: value (none) -> 0402; footprint (none) -> Resistor_SMD:R_0402_1005Metric
- R2: value (none) -> 330; footprint (none) -> Resistor_SMD:R_0805_2012Metric_Pad1.15x1.40mm_HandSolder
- R20, R21, R22, R23: value (none) -> 0603; footprint (none) -> Resistor_SMD:R_0603_1608Metric
- R24, R25, R26, R27: value (none) -> 0603HS; footprint (none) -> Resistor_SMD:R_0603_1608Metric_Pad1.05x0.95mm_HandSolder
- R28, R29, R30, R31: value (none) -> 0805; footprint (none) -> Resistor_SMD:R_0805_2012Metric
- R3: value (none) -> 330; footprint (none) -> Resistor_SMD:R_0603_1608Metric_Pad1.05x0.95mm_HandSolder
- R32, R33, R34, R35: value (none) -> 0805HS; footprint (none) -> Resistor_SMD:R_0805_2012Metric_Pad1.15x1.40mm_HandSolder
- R36, R37, R38: value (none) -> 1206; footprint (none) -> Resistor_SMD:R_1206_3216Metric
- R39, R40, R41: value (none) -> 1206HS; footprint (none) -> Resistor_SMD:R_1206_3216Metric_Pad1.42x1.75mm_HandSolder
- R4: value (none) -> 330; footprint (none) -> Resistor_SMD:R_0402_1005Metric
- R42, R43: value (none) -> 2512; footprint (none) -> Resistor_SMD:R_2512_6332Metric
- R44, R45: value (none) -> 2512HS; footprint (none) -> Resistor_SMD:R_2512_6332Metric_Pad1.52x3.35mm_HandSolder
- R5: value (none) -> 330; footprint (none) -> Resistor_SMD:R_0201_0603Metric
- TP1: value (none) -> 1206; footprint (none) -> TestPoint:TestPoint_Pad_D1.0mm
- TP2: value (none) -> 0805; footprint (none) -> TestPoint:TestPoint_Pad_D1.0mm
- TP3: value (none) -> 0603; footprint (none) -> TestPoint:TestPoint_Pad_D1.0mm
- TP4: value (none) -> 0402; footprint (none) -> TestPoint:TestPoint_Pad_D1.0mm
- TP5: value (none) -> 0201; footprint (none) -> TestPoint:TestPoint_Pad_D1.0mm
- TP6: value (none) -> ⌀1.0; footprint (none) -> TestPoint:TestPoint_Pad_D1.0mm
- TP7: value (none) -> ⌀1.5; footprint (none) -> TestPoint:TestPoint_Pad_D1.5mm
- TP8: value (none) -> ⌀2.0; footprint (none) -> TestPoint:TestPoint_Pad_D2.0mm
- U1: value (none) -> ATtiny85V-10SU; footprint (none) -> Package_SO:SOIJ-8_5.3x5.3mm_P1.27mm
- tp1: value (none) -> ⌀2.5; footprint (none) -> TestPoint:TestPoint_Pad_D2.5mm

Commit message: update
Parts:
- R26: renamed from R24; footprint Resistor_SMD:R_0603_1608Metric_Pad1.05x0.95mm_HandSolder -> Resistor_SMD:R_0603_1608Metric_Pad0.98x0.95mm_HandSolder
- R27: renamed from R32; footprint Resistor_SMD:R_0805_2012Metric_Pad1.15x1.40mm_HandSolder -> Resistor_SMD:R_0805_2012Metric_Pad1.20x1.40mm_HandSolder
- R28: renamed from R39; footprint Resistor_SMD:R_1206_3216Metric_Pad1.42x1.75mm_HandSolder -> Resistor_SMD:R_1206_3216Metric_Pad1.30x1.75mm_HandSolder
- R29: renamed from R44; footprint Resistor_SMD:R_2512_6332Metric_Pad1.52x3.35mm_HandSolder -> Resistor_SMD:R_2512_6332Metric_Pad1.40x3.35mm_HandSolder
- R31: renamed from R25; footprint Resistor_SMD:R_0603_1608Metric_Pad1.05x0.95mm_HandSolder -> Resistor_SMD:R_0603_1608Metric_Pad0.98x0.95mm_HandSolder
- R32: renamed from R33; footprint Resistor_SMD:R_0805_2012Metric_Pad1.15x1.40mm_HandSolder -> Resistor_SMD:R_0805_2012Metric_Pad1.20x1.40mm_HandSolder
- R33: renamed from R40; footprint Resistor_SMD:R_1206_3216Metric_Pad1.42x1.75mm_HandSolder -> Resistor_SMD:R_1206_3216Metric_Pad1.30x1.75mm_HandSolder
- R34: renamed from R45; footprint Resistor_SMD:R_2512_6332Metric_Pad1.52x3.35mm_HandSolder -> Resistor_SMD:R_2512_6332Metric_Pad1.40x3.35mm_HandSolder
- R36: renamed from R26; footprint Resistor_SMD:R_0603_1608Metric_Pad1.05x0.95mm_HandSolder -> Resistor_SMD:R_0603_1608Metric_Pad0.98x0.95mm_HandSolder
- R37: renamed from R34; footprint Resistor_SMD:R_0805_2012Metric_Pad1.15x1.40mm_HandSolder -> Resistor_SMD:R_0805_2012Metric_Pad1.20x1.40mm_HandSolder
- R38: renamed from R41; footprint Resistor_SMD:R_1206_3216Metric_Pad1.42x1.75mm_HandSolder -> Resistor_SMD:R_1206_3216Metric_Pad1.30x1.75mm_HandSolder
- R39: renamed from R27; footprint Resistor_SMD:R_0603_1608Metric_Pad1.05x0.95mm_HandSolder -> Resistor_SMD:R_0603_1608Metric_Pad0.98x0.95mm_HandSolder
- R40: renamed from R35; footprint Resistor_SMD:R_0805_2012Metric_Pad1.15x1.40mm_HandSolder -> Resistor_SMD:R_0805_2012Metric_Pad1.20x1.40mm_HandSolder
- R42: renamed from R2; footprint Resistor_SMD:R_0805_2012Metric_Pad1.15x1.40mm_HandSolder -> Resistor_SMD:R_0805_2012Metric_Pad1.20x1.40mm_HandSolder
- R43: renamed from R3; footprint Resistor_SMD:R_0603_1608Metric_Pad1.05x0.95mm_HandSolder -> Resistor_SMD:R_0603_1608Metric_Pad0.98x0.95mm_HandSolder
- renumbered R6 to R1, R29 to R10, R37 to R11, R43 to R12, R8 to R13, R16 to R14, R22 to R15, R30 to R16, R38 to R17, R17 to R18, R23 to R19, R14 to R2, R31 to R20, R9 to R21, R10 to R22, R18 to R23, R19 to R24, R11 to R25, R20 to R3, R12 to R30, R13 to R35, R28 to R4, R1 to R41, R4 to R44, R5 to R45, R36 to R5, R42 to R6, R15 to R8, R21 to R9, TP6 to TP1, TP7 to TP2, TP8 to TP3, tp1 to TP4, TP1 to TP5, TP2 to TP6, TP3 to TP7, TP4 to TP8, TP5 to TP9
Other:
- moved on the sheet: BT1, C1, D1, D2, D3, D4, D5, J1, R1, R10, R11, R12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

Commit message: .
Parts:
- removed Logo1: SquashedFlyLogo, SquashedFly Logo:SquashedFly Logo, symbol SquashedFly_Logo:SquashedFlyLogo
Other:
- company: Squashed Fly Ltd. -> Philip McGaw
- title: Philip McGaw's Card -> Rule
